File: STM32_AS5600_CHIPS.kicad_sch (KiCad schematic)
At the start: 39 parts, among them IC1 AS5600-ASOT, J1 Conn_01x04_Pin, J3 Conn_01x07_Pin, J4 USB4105-GF-A-120, U1 STM32F103C8Tx, U2 AMS1117-3.3, Y2 Crystal

Commit message: Add files via upload
2nd Commit
Parts:
- R7: value R -> 10k
Changed lines of the file:
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@@
 	(text "USB\n"
 		(exclude_from_sim no)
-		(at 226.568 67.056 0)
+		(at 216.662 67.056 0)
 		(effects
 			(font
@@
 			)
 		)
-		(property "Value" "R"
+		(property "Value" "10k"
 			(at 82.55 184.1499 0)
 			(effects
